File: macropad/ergogen/pcbs/switch_plate.kicad_pcb (KiCad board)
At the start: 2 copper layers, 196 x 43.9 mm, 0 parts

Commit message: More case fixes
Other:
- board size 196 x 43.9 mm -> 197 x 44.9 mm
Changed lines of the file:
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@@
   )
   (net 0 "")
-  (gr_line (start 70.7367836389337 99.95608438328529) (end 90.09061564593371 90.69587768137143) (layer Edge.Cuts) (stroke (width 0.15) (type default)))
-(gr_line (start 90.953832007 90.5) (end 144.75 90.5) (layer Edge.Cuts) (stroke (width 0.15) (type default)))
-(gr_line (start 188.45 90.5) (end 242.246167993 90.5) (layer Edge.Cuts) (stroke (width 0.15) (type default)))
-(gr_line (start 243.10938435406626 90.69587768137143) (end 262.4632163610664 99.95608438328533) (layer Edge.Cuts) (stroke (width 0.15) (type default)))
-(gr_line (start 262.4632163610664 120.04391561671466) (end 243.1093843540663 129.30412231862857) (layer Edge.Cuts) (stroke (width 0.15) (type default)))
-(gr_line (start 90.953832007 129.5) (end 144.7525016 129.5) (layer Edge.Cuts) (stroke (width 0.15) (type default)))
-(gr_line (start 188.4474984 129.5) (end 242.246167993 129.5) (layer Edge.Cuts) (stroke (width 0.15) (type default)))
-(gr_line (start 90.09061564593368 129.30412231862857) (end 70.73678363893369 120.04391561671468) (layer Edge.Cuts) (stroke (width 0.15) (type default)))
-(gr_arc (start 90.953832007 90.5) (mid 90.51125130700001 90.5495841) (end 90.090615607 90.6958776) (layer Edge.Cuts) (stroke (width 0.15) (type default)))
-(gr_arc (start 243.109384393 90.6958776) (mid 242.688748693 90.549584) (end 242.246167993 90.5) (layer Edge.Cuts) (stroke (width 0.15) (type default)))
-(gr_arc (start 262.7902548 100.15294390191387) (mid 262.6314429 100.04669400191388) (end 262.4632164 99.95608430191388) (layer Edge.Cuts) (stroke (width 0.15) (type default)))
-(gr_arc (start 262.4632164 120.04391569808611) (mid 262.6314429 119.95330599808611) (end 262.7902548 119.84705609808611) (layer Edge.Cuts) (stroke (width 0.15) (type default)))
-(gr_arc (start 242.246167993 129.5) (mid 242.688748693 129.4504159) (end 243.109384393 129.3041224) (layer Edge.Cuts) (stroke (width 0.15) (type default)))
-(gr_arc (start 90.090615607 129.3041224) (mid 90.51125130700001 129.450416) (end 90.953832007 129.5) (layer Edge.Cuts) (stroke (width 0.15) (type default)))
-(gr_arc (start 70.40974519999999 119.84705609808611) (mid 70.56855709999999 119.95330599808611) (end 70.7367836 120.04391569808611) (layer Edge.Cuts) (stroke (width 0.15) (type default)))
-(gr_arc (start 70.7367836 99.95608430191386) (mid 70.56855709999999 100.04669400191386) (end 70.40974519999999 100.15294390191386) (layer Edge.Cuts) (stroke (width 0.15) (type default)))
-(gr_line (start 144.75 90.5) (end 144.75 89.5) (layer Edge.Cuts) (stroke (width 0.15) (type default)))
-(gr_line (start 146.75 87.5) (end 186.45 87.5) (layer Edge.Cuts) (stroke (width 0.15) (type default)))
-(gr_line (start 188.45 89.5) (end 188.45 90.5) (layer Edge.Cuts) (stroke (width 0.15) (type default)))
-(gr_line (start 186.45 131.4) (end 146.75 131.4) (layer Edge.Cuts) (stroke (width 0.15) (type default)))
-(gr_arc (start 146.75 87.5) (mid 145.3357864 88.0857864) (end 144.75 89.5) (layer Edge.Cuts) (stroke (width 0.15) (type default)))
-(gr_arc (start 188.45 89.5) (mid 187.8642136 88.0857864) (end 186.45 87.5) (layer Edge.Cuts) (stroke (width 0.15) (type default)))
-(gr_arc (start 186.45 131.4) (mid 187.82840489999998 130.8491377) (end 188.4474984 129.5) (layer Edge.Cuts) (stroke (width 0.15) (type default)))
-(gr_arc (start 144.7525016 129.5) (mid 145.3715951 130.8491376) (end 146.75 131.4) (layer Edge.Cuts) (stroke (width 0.15) (type default)))
-(gr_arc (start 70.40974519999999 100.152944) (mid 69.08140519999999 101.5975042) (end 68.6 103.5) (layer Edge.Cuts) (stroke (width 0.15) (type default)))
-(gr_line (start 68.6 103.5) (end 68.6 116.5) (layer Edge.Cuts) (stroke (width 0.15) (type default)))
-(gr_arc (start 68.6 116.5) (mid 69.08140519999999 118.4024958) (end 70.40974519999999 119.847056) (layer Edge.Cuts) (stroke (width 0.15) (type default)))
-(gr_arc (start 262.7902548 119.847056) (mid 264.11859480000004 118.4024958) (end 264.6 116.5) (layer Edge.Cuts) (stroke (width 0.15) (type default)))
-(gr_line (start 264.6 116.5) (end 264.6 103.5) (layer Edge.Cuts) (stroke (width 0.15) (type default)))
-(gr_arc (start 264.6 103.5) (mid 264.11859480000004 101.5975042) (end 262.7902548 100.152944) (layer Edge.Cuts) (stroke (width 0.15) (type default)))
+  (gr_line (start 70.5212648 99.50491730191386) (end 89.87452630700001 90.2449836) (layer Edge.Cuts) (stroke (width 0.15) (type default)))
+(gr_arc (start 90.953832007 90) (mid 90.400606207 90.0619801) (end 89.874811507 90.2448471) (layer Edge.Cuts) (stroke (width 0.15) (type default)))
+(gr_line (start 90.953832007 90) (end 144.25 90) (layer Edge.Cuts) (stroke (width 0.15) (type default)))
+(gr_line (start 144.25 90) (end 144.25 89.5) (layer Edge.Cuts) (stroke (width 0.15) (type default)))
+(gr_arc (start 146.75 87) (mid 144.982233 87.732233) (end 144.25 89.5) (layer Edge.Cuts) (stroke (width 0.15) (type default)))
+(gr_line (start 146.75 87) (end 186.45 87) (layer Edge.Cuts) (stroke (width 0.15) (type default)))
+(gr_arc (start 188.95 89.5) (mid 188.21776699999998 87.732233) (end 186.45 87) (layer Edge.Cuts) (stroke (width 0.15) (type default)))
+(gr_line (start 188.95 89.5) (end 188.95 90) (layer Edge.Cuts) (stroke (width 0.15) (type default)))
+(gr_line (start 188.95 90) (end 242.246167993 90) (layer Edge.Cuts) (stroke (width 0.15) (type default)))
+(gr_arc (start 243.325188493 90.2448471) (mid 242.799393893 90.0619801) (end 242.246167993 90) (layer Edge.Cuts) (stroke (width 0.15) (type default)))
+(gr_line (start 243.325473693 90.2449836) (end 262.6787352 99.50491730191388) (layer Edge.Cuts) (stroke (width 0.15) (type default)))
+(gr_arc (start 263.0758354 99.74230930191388) (mid 262.8829243 99.61448880191388) (end 262.67902050000004 99.50505370191388) (layer Edge.Cuts) (stroke (width 0.15) (type default)))
+(gr_arc (start 265.1 103.5) (mid 264.561771 101.3659029) (end 263.0758353 99.7423093) (layer Edge.Cuts) (stroke (width 0.15) (type default)))
+(gr_line (start 265.1 116.5) (end 265.1 103.5) (layer Edge.Cuts) (stroke (width 0.15) (type default)))
+(gr_arc (start 263.0758353 120.2576907) (mid 264.561771 118.6340971) (end 265.1 116.5) (layer Edge.Cuts) (stroke (width 0.15) (type default)))
+(gr_arc (start 262.67902050000004 120.49494619808611) (mid 262.8829243 120.3855111980861) (end 263.0758354 120.25769059808611) (layer Edge.Cuts) (stroke (width 0.15) (type default)))
+(gr_line (start 262.6787352 120.49508269808611) (end 243.325473693 129.75501640000002) (layer Edge.Cuts) (stroke (width 0.15) (type default)))
+(gr_arc (start 242.246167993 130) (mid 242.799393793 129.9380199) (end 243.325188493 129.7551529) (layer Edge.Cuts) (stroke (width 0.15) (type default)))
+(gr_line (start 188.8769322 130) (end 242.246167993 130) (layer Edge.Cuts) (stroke (width 0.15) (type default)))
+(gr_arc (start 186.45 131.9) (mid 187.99110349999998 131.368502) (end 188.8769322 130) (layer Edge.Cuts) (stroke (width 0.15) (type default)))
+(gr_line (start 186.45 131.9) (end 146.75 131.9) (layer Edge.Cuts) (stroke (width 0.15) (type default)))
+(gr_arc (start 144.3230678 130) (mid 145.2088965 131.368502) (end 146.75 131.9) (layer Edge.Cuts) (stroke (width 0.15) (type default)))
+(gr_line (start 90.953832007 130) (end 144.3230678 130) (layer Edge.Cuts) (stroke (width 0.15) (type default)))
+(gr_arc (start 89.874811507 129.7551529) (mid 90.400606107 129.9380199) (end 90.953832007 130) (layer Edge.Cuts) (stroke (width 0.15) (type default)))
+(gr_line (start 89.87452630700001 129.75501640000002) (end 70.5212648 120.49508269808611) (layer Edge.Cuts) (stroke (width 0.15) (type default)))
+(gr_arc (start 70.1241646 120.25769069808611) (mid 70.31707569999999 120.3855111980861) (end 70.5209795 120.49494629808612) (layer Edge.Cuts) (stroke (width 0.15) (type default)))
+(gr_arc (start 68.1 116.5) (mid 68.638229 118.6340971) (end 70.1241647 120.2576907) (layer Edge.Cuts) (stroke (width 0.15) (type default)))
+(gr_line (start 68.1 103.5) (end 68.1 116.5) (layer Edge.Cuts) (stroke (width 0.15) (type default)))
+(gr_arc (start 70.1241647 99.7423093) (mid 68.638229 101.3659029) (end 68.1 103.5) (layer Edge.Cuts) (stroke (width 0.15) (type default)))
+(gr_arc (start 70.5209795 99.50505380191386) (mid 70.31707569999999 99.61448880191386) (end 70.1241646 99.74230940191386) (layer Edge.Cuts) (stroke (width 0.15) (type default)))
 (gr_line (start 93 127) (end 107 127) (layer Edge.Cuts) (stroke (width 0.15) (type default)))
 (gr_line (start 107 127) (end 107 113) (layer Edge.Cuts) (stroke (width 0.15) (type default)))
