File: pekeboard/pcbs/pepekey.kicad_pcb (KiCad board)
At the start: 2 copper layers, 148.2 x 123.9 mm, 63 parts

Commit message: updating generated files
Routing:
- net P011: track 248.8 -> 259.5 mm
- net RST: track 47.5 -> 41.6 mm, vias 0 -> 1
- net P115: track 169.0 -> 163.4 mm, vias 6 -> 8
- net P100: track 257.9 -> 262.9 mm
- net outer_num: track 28.0 -> 32.6 mm
- net outer_bottom: track 32.6 -> 28.0 mm
- net P024: track 231.2 -> 227.1 mm
- net outer_thumbrow: track 34.4 -> 30.3 mm
- net outer_top: track 28.6 -> 32.1 mm
- net ring_num: track 28.6 -> 31.8 mm
- net P022: track 247.5 -> 244.5 mm
- net P002: track 163.3 -> 166.3 mm
- net inner_top: track 31.9 -> 29.5 mm
- net pinky_home: track 30.4 -> 28.3 mm
- net ring_home: track 28.4 -> 30.3 mm, vias 2 -> 3
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Other:
- rule pad_to_mask_clearance: 0 -> 0.05
