File: pekeboard/pcbs/pepekey_l.kicad_pcb (KiCad board)
At the start: 2 copper layers, 148.2 x 123.9 mm, 63 parts

Commit message: submodule ref
Routing:
- net P031: track 164.0 -> 185.4 mm, vias 4 -> 2
- net P022: track 179.5 -> 167.2 mm, vias 1 -> 2
- net P113: track 137.4 -> 128.2 mm, vias 2 -> 0
- net P024: track 142.2 -> 151.5 mm, vias 1 -> 2
- net P106: track 111.8 -> 118.9 mm
- net P115: track 156.1 -> 154.1 mm, vias 6 -> 5
- net P008: track 186.1 -> 184.8 mm
- net outer_home: track 13.0 -> 12.3 mm, vias 1 -> 0
- net P100: track 123.6 -> 122.9 mm, vias 1 -> 2
- net GND: track 67.9 -> 67.4 mm
- net inner_thumbrow: track 12.3 -> 11.9 mm, vias 1 -> 0
- net P002: track 162.9 -> 162.5 mm, vias 5 -> 4
- net P111: track 80.9 -> 80.7 mm, vias 1 -> 0
- net P011: track 129.3 -> 129.4 mm, vias 1 -> 2
- net outer_num: track 12.4 -> 12.3 mm, vias 1 -> 0
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Other:
- board size 148.2 x 123.9 mm -> 148.5 x 124.9 mm
- board text added: "Pekeboard v1.0 by pedroren"
