File: pekeboard/pcbs/pepekey_r.kicad_pcb (KiCad board)
At the start: 2 copper layers, 148.2 x 123.9 mm, 63 parts

Commit message: submodule ref
Routing:
- net P113: track 44.6 -> 126.6 mm
- net P115: track 132.2 -> 150.4 mm
- net P106: track 124.0 -> 131.0 mm
- net P031: track 179.2 -> 173.0 mm, vias 4 -> 3
- net RAW: track 50.6 -> 44.7 mm
- net P024: track 144.9 -> 150.8 mm
- net P002: track 135.5 -> 141.3 mm
- net P008: track 203.1 -> 207.6 mm
- net GND: track 62.4 -> 64.2 mm
- net P100: track 124.2 -> 125.5 mm
- net P029: vias 7 -> 5
Other:
- board size 148.2 x 123.9 mm -> 148.5 x 124.9 mm
- board text added: "Pekeboard v1.0 by pedroren"
