File: pekeboard/pcbs/bottom_plate.kicad_pcb (KiCad board)
At the start: 2 copper layers, 148.5 x 124.9 mm, 0 parts

Commit message: cleanup and built zmk firmware files
Other:
- outline, holes or cut-outs redrawn
Changed lines of the file:
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@@
   (title_block
     (title "bottom_plate")
-    (date "2026-06-12")
+    (date "2026-06-27")
     (rev "1")
     (company "pedroren")
@@
 (gr_line (start 220.71276159999996 129.8613317) (end 220.57536534191308 129.29632909913016) (layer Edge.Cuts) (stroke (width 0.15) (type default)))
 (gr_line (start 220.40174753758978 128.83724882936644) (end 219.25665352191666 126.6620800546259) (layer Edge.Cuts) (stroke (width 0.15) (type default)))
-(gr_line (start 218.17094725531445 125.71435866370682) (end 210.3663004500163 122.87369953625407) (layer Edge.Cuts) (stroke (width 0.15) (type default)))
-(gr_line (start 209.05054856169332 120.96547870555514) (end 209.0547370565438 120.67499999999927) (layer Edge.Cuts) (stroke (width 0.15) (type default)))
+(gr_line (start 209.4516831456666 93.14616440144164) (end 209.4581718233103 92.69616440144273) (layer Edge.Cuts) (stroke (width 0.15) (type default)))
 (gr_arc (start 191.05139831664007 141.5949006501004) (mid 191.00579051664008 141.57942735010042) (end 190.95982331664007 141.5650568501004) (layer Edge.Cuts) (stroke (width 0.15) (type default)))
 (gr_arc (start 220.57536535928972 129.2963290705867) (mid 220.5026925592897 129.0614428705867) (end 220.4017475592897 128.8372487705867) (layer Edge.Cuts) (stroke (width 0.15) (type default)))
-(gr_arc (start 219.25665354361664 126.66208009584622) (mid 218.80212994361665 126.08702939584622) (end 218.17094734361663 125.71435859584622) (layer Edge.Cuts) (stroke (width 0.15) (type default)))
-(gr_arc (start 209.0505485617141 120.96547870411469) (mid 209.40380926171412 122.12962670411468) (end 210.3663004617141 122.87369950411468) (layer Edge.Cuts) (stroke (width 0.15) (type default)))
-(gr_line (start 235.02500000000003 118.675) (end 235.02500000000003 45.57500000000001) (layer Edge.Cuts) (stroke (width 0.15) (type default)))
+(gr_arc (start 219.25665354361664 126.66208009584622) (mid 219.09516144361663 126.40482919584622) (end 218.89657574361664 126.17499999584622) (layer Edge.Cuts) (stroke (width 0.15) (type default)))
+(gr_line (start 211.45796392333108 90.72500000000001) (end 233.02500000000003 90.72500000000001) (layer Edge.Cuts) (stroke (width 0.15) (type default)))
+(gr_arc (start 233.02500000000003 90.72500000000001) (mid 234.43921360000004 90.1392136) (end 235.02500000000003 88.72500000000001) (layer Edge.Cuts) (stroke (width 0.15) (type default)))
+(gr_line (start 235.02500000000003 88.72500000000001) (end 235.02500000000003 45.57500000000001) (layer Edge.Cuts) (stroke (width 0.15) (type default)))
 (gr_arc (start 235.02500000000003 45.57500000000001) (mid 234.43921360000004 44.160786400000006) (end 233.02500000000003 43.57500000000001) (layer Edge.Cuts) (stroke (width 0.15) (type default)))
 (gr_line (start 233.02500000000003 43.575) (end 206.57500000000002 43.575) (layer Edge.Cuts) (stroke (width 0.15) (type default)))
 (gr_arc (start 206.57500000000002 43.575) (mid 206.01511380000002 43.654966800000004) (end 205.50000000000003 43.888472500000006) (layer Edge.Cuts) (stroke (width 0.15) (type default)))
-(gr_line (start 209.0547370565438 120.675) (end 233.02500000000003 120.675) (layer Edge.Cuts) (stroke (width 0.15) (type default)))
-(gr_arc (start 233.02500000000003 120.675) (mid 234.43921360000004 120.0892136) (end 235.02500000000003 118.675) (layer Edge.Cuts) (stroke (width 0.15) (type default)))
+(gr_line (start 218.89657574361664 126.17499999584622) (end 233.02500000000003 126.175) (layer Edge.Cuts) (stroke (width 0.15) (type default)))
+(gr_arc (start 233.02500000000003 126.175) (mid 234.43921360000004 125.5892136) (end 235.02500000000003 124.175) (layer Edge.Cuts) (stroke (width 0.15) (type default)))
+(gr_line (start 235.02500000000003 124.175) (end 235.02500000000003 97.175) (layer Edge.Cuts) (stroke (width 0.15) (type default)))
+(gr_arc (start 235.02500000000003 97.175) (mid 234.43921360000004 95.7607864) (end 233.02500000000003 95.175) (layer Edge.Cuts) (stroke (width 0.15) (type default)))
+(gr_line (start 233.02500000000003 95.175) (end 211.45147524568742 95.175) (layer Edge.Cuts) (stroke (width 0.15) (type default)))
+(gr_arc (start 209.4516831456874 93.1461644) (mid 210.0271032456874 94.57898159999999) (end 211.45147524568742 95.175) (layer Edge.Cuts) (stroke (width 0.15) (type default)))
+(gr_arc (start 211.45796392333108 90.72500000000036) (mid 210.05398232333107 91.30062800000036) (end 209.45817182333107 92.69616440000037) (layer Edge.Cuts) (stroke (width 0.15) (type default)))
 (gr_circle (center 129.5 58.25) (end 131 58.25) (layer Edge.Cuts) (stroke (width 0.15) (type default)) (fill none))
 (gr_circle (center 128.5 110.5) (end 130 110.5) (layer Edge.Cuts) (stroke (width 0.15) (type default)) (fill none))
@@
 (gr_circle (center 181.7 117.15) (end 183.2 117.15) (layer Edge.Cuts) (stroke (width 0.15) (type default)) (fill none))
 (gr_circle (center 215.73751329999996 135.53425919999998) (end 217.23751329999996 135.53425919999998) (layer Edge.Cuts) (stroke (width 0.15) (type default)) (fill none))
-(gr_circle (center 230.95000000000002 93.2) (end 232.45000000000002 93.2) (layer Edge.Cuts) (stroke (width 0.15) (type default)) (fill none))
 )
